File: 2025-08-02-multi-test-pcb/2025-08-02-multi-test-pcb.kicad_sch (KiCad schematic)
At the start: 7 parts, among them J1 Conn_02x15_Odd_Even, SW1 SW_SPDT

Commit message: wip
Parts:
- added SW2: RotaryEncoder_Switch_RG, Input:RotaryEncoder_Switch_RG, symbol Input:RotaryEncoder_Switch_RG
- added SW3: RotaryEncoder_Switch_RGB, Input:RotaryEncoder_Switch_RGB, symbol Input:RotaryEncoder_Switch_RGB
- added U2: ~, Modules:AliE_MP1584EN_regulator, symbol Modules:AliE_MP1584EN_regulator
- added U3: RS485 to TTL module, Modules:RS485_to_ttl, symbol Modules:RS485_to_TTL

Commit message: wip
Parts:
- added D1: D_Schottky, symbol Device:D_Schottky
- added J2: Conn_01x02, Connectors:CTB7000-2, symbol Connector_Generic:Conn_01x02
- added J3: Conn_01x03, Connectors:CTB7000-3, symbol Connector_Generic:Conn_01x03
- added J4, J5: Conn_01x03, Connector_PinHeader_2.54mm:PinHeader_1x03_P2.54mm_Vertical, symbol Connector_Generic:Conn_01x03
- added J6: Conn_01x05, Connector_PinHeader_2.54mm:PinHeader_1x05_P2.54mm_Vertical, symbol Connector_Generic:Conn_01x05
- added J7: Conn_01x04, Connector_PinHeader_2.54mm:PinHeader_1x04_P2.54mm_Vertical, symbol Connector_Generic:Conn_01x04
- added J8: Conn_01x06, Connector_PinHeader_2.54mm:PinHeader_1x06_P2.54mm_Vertical, symbol Connector_Generic:Conn_01x06
- SW1: footprint (none) -> Input:AliE_SPDT_Lever_Switch
- U2: value ~ -> 5V
Connections:
- net +3.3V: now also SW3.5 (VIN), U3.1 (VCC), J4.2 (Pin_2), J8.3 (Pin_3)
- net +5V: now also D1.1 (K), J4.3 (Pin_3)
- net GND: now also SW2.1 (GND), SW2.C, SW3.C, U2.4 (GND), U3.4 (GND), J4.1 (Pin_1), J8.1 (Pin_1)
- net IO_16: now also U3.2 (TXD), J8.4 (Pin_4)
- net IO_17: now also U3.3 (RXD), J8.5 (Pin_5)
- net at SW1.1 (A): now also J5.1 (Pin_1)
- net at SW1.2 (B): now also J5.2 (Pin_2)
- net at SW1.3 (C): now also J5.3 (Pin_3)
- net at U3.5 (A+): now also J3.1 (Pin_1)
- net at U3.6 (B-): now also J3.2 (Pin_2)
- net at U3.7 (BUS_GND): now also J3.3 (Pin_3)
- net at U2.1 (VIN): now also J2.2 (Pin_2)
- net at U2.2 (GND): now also J2.1 (Pin_1)
- net at U2.3 (VOUT): now also D1.2 (A)
- no-connect marks 4 -> 24
Other:
- moved on the sheet: SW1, SW2, SW3, U2, U3

Commit message: wip
Parts:
- D1: footprint (none) -> Diode_SMD:D_SOD-123
Connections:
- net at J6.1 (Pin_1): now also SW3.B
- net at J6.2 (Pin_2): now also SW3.A
- net at J7.1 (Pin_1): now also SW2.B
- net at J7.2 (Pin_2): now also SW2.A
Changed lines of the file:
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@@
 	(wire
 		(pts
+			(xy 182.88 48.26) (xy 173.99 48.26)
+		)
+		(stroke
+			(width 0)
+			(type default)
+		)
+	)
+	(wire
+		(pts
 			(xy 109.22 91.44) (xy 111.76 91.44)
 		)
@@
 	(wire
 		(pts
+			(xy 180.34 60.96) (xy 194.31 60.96)
+		)
+		(stroke
+			(width 0)
+			(type default)
+		)
+	)
+	(wire
+		(pts
 			(xy 209.55 134.62) (xy 222.25 134.62)
 		)
@@
 	(wire
 		(pts
+			(xy 180.34 53.34) (xy 180.34 60.96)
+		)
+		(stroke
+			(width 0)
+			(type default)
+		)
+	)
+	(wire
+		(pts
 			(xy 184.15 127) (xy 196.85 127)
 		)
@@
 	(wire
 		(pts
+			(xy 224.79 48.26) (xy 233.68 48.26)
+		)
+		(stroke
+			(width 0)
+			(type default)
+		)
+	)
+	(wire
+		(pts
 			(xy 209.55 124.46) (xy 222.25 124.46)
 		)
@@
 	(wire
 		(pts
+			(xy 173.99 48.26) (xy 173.99 62.23)
+		)
+		(stroke
+			(width 0)
+			(type default)
+		)
+	)
+	(wire
+		(pts
 			(xy 152.4 86.36) (xy 154.94 86.36)
 		)
@@
 	(wire
 		(pts
+			(xy 173.99 62.23) (xy 191.77 62.23)
+		)
+		(stroke
+			(width 0)
+			(type default)
+		)
+	)
+	(wire
+		(pts
 			(xy 38.1 133.35) (xy 40.64 133.35)
 		)
@@
 	(wire
 		(pts
+			(xy 243.84 62.23) (xy 224.79 62.23)
+		)
+		(stroke
+			(width 0)
+			(type default)
+		)
+	)
+	(wire
+		(pts
+			(xy 224.79 62.23) (xy 224.79 48.26)
+		)
+		(stroke
+			(width 0)
+			(type default)
+		)
+	)
+	(wire
+		(pts
+			(xy 182.88 53.34) (xy 180.34 53.34)
+		)
+		(stroke
+			(width 0)
+			(type default)
+		)
+	)
+	(wire
+		(pts
 			(xy 184.15 132.08) (xy 196.85 132.08)
 		)
@@
 	(wire
 		(pts
+			(xy 246.38 60.96) (xy 246.38 63.5)
+		)
+		(stroke
+			(width 0)
+			(type default)
+		)
+	)
+	(wire
+		(pts
 			(xy 71.12 128.27) (xy 73.66 128.27)
 		)
@@
 	(wire
 		(pts
+			(xy 233.68 53.34) (xy 231.14 53.34)
+		)
+		(stroke
+			(width 0)
+			(type default)
+		)
+	)
+	(wire
+		(pts
 			(xy 71.12 125.73) (xy 73.66 125.73)
 		)
@@
 	(wire
 		(pts
+			(xy 194.31 60.96) (xy 194.31 63.5)
+		)
+		(stroke
+			(width 0)
+			(type default)
+		)
+	)
+	(wire
+		(pts
 			(xy 209.55 142.24) (xy 233.68 142.24)
 		)
@@
 	(wire
 		(pts
+			(xy 243.84 63.5) (xy 243.84 62.23)
+		)
+		(stroke
+			(width 0)
+			(type default)
+		)
+	)
+	(wire
+		(pts
 			(xy 209.55 127) (xy 222.25 127)
 		)
@@
 	(wire
 		(pts
+			(xy 231.14 60.96) (xy 246.38 60.96)
+		)
+		(stroke
+			(width 0)
+			(type default)
+		)
+	)
+	(wire
+		(pts
 			(xy 184.15 134.62) (xy 196.85 134.62)
 		)
@@
 		)
 	)
+	(wire
+		(pts
+			(xy 191.77 62.23) (xy 191.77 63.5)
+		)
+		(stroke
+			(width 0)
+			(type default)
+		)
+	)
+	(wire
+		(pts
+			(xy 231.14 53.34) (xy 231.14 60.96)
+		)
+		(stroke
+			(width 0)
+			(type default)
+		)
+	)
 	(label "IO_20"
 		(at 222.25 132.08 0)
@@
 			)
 		)
-		(property "Footprint" ""
+		(property "Footprint" "Diode_SMD:D_SOD-123"
 			(at 148.59 86.36 0)
 			(effects

Commit message: wip
Parts:
- removed J5: Conn_01x03, Connector_PinHeader_2.54mm:PinHeader_1x03_P2.54mm_Vertical, symbol Connector_Generic:Conn_01x03
- removed J6: Conn_01x05, Connector_PinHeader_2.54mm:PinHeader_1x05_P2.54mm_Vertical, symbol Connector_Generic:Conn_01x05
- removed J7: Conn_01x04, Connector_PinHeader_2.54mm:PinHeader_1x04_P2.54mm_Vertical, symbol Connector_Generic:Conn_01x04
- added J5: Conn_02x07_Odd_Even, Connector_PinHeader_2.54mm:PinHeader_2x07_P2.54mm_Vertical, symbol Connector_Generic:Conn_02x07_Odd_Even
Connections:
- net GND: now also SW1.2 (B)
- net SW_1: now reaches SW1.1 (A)
- net SW_1: now also J5.12 (Pin_12)
- net SW_2: now reaches SW1.3 (C)
- net SW_2: now also J5.14 (Pin_14)
- net ENC_1_B: now reaches SW3.B
- net ENC_1_B: now also J5.1 (Pin_1)
- net ENC_1_A: now reaches SW3.A
- net ENC_1_A: now also J5.3 (Pin_3)
- net ENC_1_LR: now reaches SW3.1 (R)
- net ENC_1_LR: now also J5.11 (Pin_11)
- net ENC_1_LG: now reaches SW3.2 (G)
- net ENC_1_LG: now also J5.9 (Pin_9)
- net ENC_1_SW: now reaches SW3.3 (SW)
- net ENC_1_SW: now also J5.7 (Pin_7)
- net ENC_1_LB: now reaches SW3.4 (B)
- net ENC_1_LB: now also J5.5 (Pin_5)
- net ENC_2_B: now reaches SW2.B
- net ENC_2_B: now also J5.10 (Pin_10)
- net ENC_2_A: now reaches SW2.A
- net ENC_2_A: now also J5.8 (Pin_8)
- net ENC_2_LR: now reaches SW2.2 (R)
- net ENC_2_LR: now also J5.6 (Pin_6)
- net ENC_2_LG: now reaches SW2.3 (G)
- net ENC_2_LG: now also J5.4 (Pin_4)
- net ENC_2_SW: now reaches SW2.4 (SW)
- net ENC_2_SW: now also J5.2 (Pin_2)
Other:
- moved on the sheet: SW1, SW2
