File: 2025-08-02-multi-test-pcb/2025-08-02-multi-test-pcb.kicad_pcb (KiCad board)
At the start: 2 copper layers, 102.9 x 53.3 mm, 6 parts, among them J1 Conn_02x15_Odd_Even

Commit message: wip
Parts:
- added SW2: RotaryEncoder_Switch_RG, Input:RotaryEncoder_Switch_RG, F.Cu at (144.8, 85.0)
- added SW3: RotaryEncoder_Switch_RGB, Input:RotaryEncoder_Switch_RGB, F.Cu at (160.0, 85.0)
- added U1: ~, Displays:ILI9341_2.8in_with_touch_and_sd, F.Cu at (127.0, 101.0)
- added U2: ~, Modules:AliE_MP1584EN_regulator, F.Cu at (106.0, 95.0)
- added U3: RS485 to TTL module, Modules:RS485_to_ttl, B.Cu at (105.5, 102.0)

Commit message: wip
Parts:
- removed REF**: OSHW-Logo2_9.8x8mm_SilkScreen, Symbol:OSHW-Logo2_9.8x8mm_SilkScreen
- added J2: Conn_01x02, Connectors:CTB7000-2, B.Cu at (94.6, 121.9)
- added J3: Conn_01x03, Connectors:CTB7000-3, B.Cu at (92.1, 78.7)
- added J4: Conn_01x03, Connector_PinHeader_2.54mm:PinHeader_1x03_P2.54mm_Vertical, F.Cu at (129.5, 78.0)
- added J5: Conn_01x03, Connector_PinHeader_2.54mm:PinHeader_1x03_P2.54mm_Vertical, F.Cu at (152.4, 113.7)
- added J6: Conn_01x05, Connector_PinHeader_2.54mm:PinHeader_1x05_P2.54mm_Vertical, F.Cu at (160.7, 96.5)
- added J7: Conn_01x04, Connector_PinHeader_2.54mm:PinHeader_1x04_P2.54mm_Vertical, F.Cu at (144.1, 96.5)
- added J8: Conn_01x06, Connector_PinHeader_2.54mm:PinHeader_1x06_P2.54mm_Vertical, F.Cu at (120.7, 124.0)
- added SW1: SW_SPDT, Input:AliE_SPDT_Lever_Switch, F.Cu at (152.4, 101.9)
- U2: value ~ -> 5V
- moved U2 10.6 mm to (108.0, 105.4), turned to 0 degrees
- moved U3 2.46 mm to (108.0, 102.2)
- moved SW2 0.66 mm to (144.1, 85.0)
- moved SW3 0.66 mm to (160.7, 85.0)
Connections:
- SW2 pad 1: unconnected-(SW2-GND-Pad1) -> GND
- SW2 pad C: unconnected-(SW2-PadC) -> GND
- SW3 pad 5: unconnected-(SW3-VIN-Pad5) -> +3.3V
- SW3 pad C: unconnected-(SW3-PadC) -> GND
- U2 pad 1: unconnected-(U2-VIN-Pad1) -> Net-(J2-Pin_2)
- U2 pad 2: unconnected-(U2-GND-Pad2) -> Net-(J2-Pin_1)
- U2 pad 3: unconnected-(U2-VOUT-Pad3) -> Net-(D1-A)
- U2 pad 4: unconnected-(U2-GND-Pad4) -> GND
- U3 pad 1: unconnected-(U3-VCC-Pad1) -> +3.3V
- U3 pad 2: unconnected-(U3-TXD-Pad2) -> /IO_16
- U3 pad 3: unconnected-(U3-RXD-Pad3) -> /IO_17
- U3 pad 4: unconnected-(U3-GND-Pad4) -> GND
- U3 pad 5: unconnected-(U3-A+-Pad5) -> Net-(J3-Pin_1)
- U3 pad 6: unconnected-(U3-B--Pad6) -> Net-(J3-Pin_2)
- U3 pad 7: unconnected-(U3-BUS_GND-Pad7) -> Net-(J3-Pin_3)
Other:
- board text removed: "2025-07-23"
- board text removed: "dan-nixon.com"
- board text removed: "github.com/DanNixon/peek-o-display"

Commit message: wip
Parts:
- added D1: D_Schottky, Diode_SMD:D_SOD-123, F.Cu at (119.4, 90.2)
- moved J5 5.08 mm to (152.4, 118.7), turned to 180 degrees
- moved J4 1.27 mm to (130.8, 78.0)
Routing:
- net +3.3V: track 0.00 -> 111.7 mm
- net /IO_17: track 0.00 -> 41.8 mm
- net /IO_16: track 0.00 -> 33.9 mm
- net Net-(J2-Pin_1): track 0.00 -> 25.9 mm
- net Net-(J5-Pin_1): track 0.00 -> 23.8 mm
- net Net-(D1-A): track 0.00 -> 21.1 mm
- net Net-(J3-Pin_2): track 0.00 -> 19.6 mm
- net Net-(J3-Pin_1): track 0.00 -> 18.5 mm
- net Net-(J3-Pin_3): track 0.00 -> 17.5 mm
- net Net-(J5-Pin_2): track 0.00 -> 16.0 mm
- net +5V: track 0.00 -> 13.4 mm
- net Net-(J2-Pin_2): track 0.00 -> 12.8 mm
- net Net-(J5-Pin_3): track 0.00 -> 7.11 mm

Commit message: wip
Parts:
- removed J6: Conn_01x05, Connector_PinHeader_2.54mm:PinHeader_1x05_P2.54mm_Vertical
- removed J7: Conn_01x04, Connector_PinHeader_2.54mm:PinHeader_1x04_P2.54mm_Vertical
- J5: value Conn_01x03 -> Conn_02x07_Odd_Even; footprint Connector_PinHeader_2.54mm:PinHeader_1x03_P2.54mm_Vertical -> Connector_PinHeader_2.54mm:PinHeader_2x07_P2.54mm_Vertical
- moved J5 20.1 mm to (146.0, 99.7), turned to 0 degrees
- moved SW3 16.5 mm to (144.1, 85.1)
- moved SW2 16.5 mm to (160.7, 85.0)
- moved SW1 14.8 mm to (159.4, 114.9)
Connections:
- J5 pad 1: Net-(J5-Pin_1) -> /ENC_1_B
- J5 pad 2: Net-(J5-Pin_2) -> /ENC_2_SW
- J5 pad 3: Net-(J5-Pin_3) -> /ENC_1_A
- SW1 pad 1: Net-(J5-Pin_1) -> /SW_1
- SW1 pad 2: Net-(J5-Pin_2) -> GND
- SW1 pad 3: Net-(J5-Pin_3) -> /SW_2
- SW2 pad 2: unconnected-(SW2-R-Pad2) -> /ENC_2_LR
- SW2 pad 3: unconnected-(SW2-G-Pad3) -> /ENC_2_LG
- SW2 pad 4: unconnected-(SW2-SW-Pad4) -> /ENC_2_SW
- SW2 pad A: unconnected-(SW2-PadA) -> /ENC_2_A
- SW2 pad B: unconnected-(SW2-PadB) -> /ENC_2_B
- SW3 pad 1: unconnected-(SW3-R-Pad1) -> /ENC_1_LR
- SW3 pad 2: unconnected-(SW3-G-Pad2) -> /ENC_1_LG
- SW3 pad 3: unconnected-(SW3-SW-Pad3) -> /ENC_1_SW
- SW3 pad 4: unconnected-(SW3-B-Pad4) -> /ENC_1_LB
- SW3 pad A: unconnected-(SW3-PadA) -> /ENC_1_A
- SW3 pad B: unconnected-(SW3-PadB) -> /ENC_1_B
Routing:
- net /ENC_1_LR: track 0.00 -> 38.1 mm
- net /ENC_1_LG: track 0.00 -> 35.4 mm
- net /ENC_1_SW: track 0.00 -> 33.1 mm
- net /ENC_2_LR: track 0.00 -> 32.2 mm
- net /ENC_2_LG: track 0.00 -> 29.3 mm
- net /ENC_1_LB: track 0.00 -> 28.8 mm
- net /ENC_2_SW: track 0.00 -> 25.5 mm
- net Net-(J5-Pin_1): track 23.8 -> 0.00 mm
- net /ENC_2_B: track 0.00 -> 23.4 mm
- net /ENC_2_A: track 0.00 -> 18.8 mm
- net +3.3V: track 111.7 -> 95.2 mm
- net Net-(J5-Pin_2): track 16.0 -> 0.00 mm
- net /SW_2: track 0.00 -> 12.7 mm
- net /SW_1: track 0.00 -> 11.7 mm
- net /ENC_1_A: track 0.00 -> 11.5 mm
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Other:
- board text added: "A"
- board text added: "B"
- board text added: "G"
- board text added: "VIN"

Commit message: wip
Routing:
- net +3.3V: track 95.2 -> 98.9 mm
- net GND: vias 0 -> 1
Changed lines of the file:
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@@
 		(at 107.95 102.235 90)
 		(property "Reference" "U3"
-			(at -20.5 -8.5 -270)
+			(at -20.5 -8.5 90)
 			(unlocked yes)
 			(layer "B.Fab")
@@
 		)
 	)
+	(via
+		(at 132.08 121.92)
+		(size 0.6)
+		(drill 0.3)
+		(layers "F.Cu" "B.Cu")
+		(free yes)
+		(net 4)
+	)
 	(segment
 		(start 106.693957 122.331703)
@@
 	)
 	(segment
+		(start 133.82676 125.151)
+		(end 134.62 124.35776)
+		(width 0.2)
+		(layer "F.Cu")
+		(net 18)
+	)
+	(segment
 		(start 148.145 78.09)
 		(end 146.904 76.849)
-		(width 0.2)
-		(layer "F.Cu")
-		(net 18)
-	)
-	(segment
-		(start 125.73 124)
-		(end 126.881 125.151)
 		(width 0.2)
 		(layer "F.Cu")
@@
 	)
 	(segment
-		(start 131.961 119.311)
-		(end 128.25 115.6)
-		(width 0.2)
-		(layer "F.Cu")
-		(net 18)
-	)
-	(segment
-		(start 126.881 125.151)
-		(end 131.28676 125.151)
-		(width 0.2)
-		(layer "F.Cu")
-		(net 18)
-	)
-	(segment
 		(start 129.421 76.849)
 		(end 128.27 78)
+		(width 0.2)
+		(layer "F.Cu")
+		(net 18)
+	)
+	(segment
+		(start 125.73 124)
+		(end 126.881 125.151)
 		(width 0.2)
 		(layer "F.Cu")
@@
 	)
 	(segment
+		(start 134.62 124.35776)
+		(end 134.62 121.97)
+		(width 0.2)
+		(layer "F.Cu")
+		(net 18)
+	)
+	(segment
+		(start 134.62 121.97)
+		(end 128.25 115.6)
+		(width 0.2)
+		(layer "F.Cu")
+		(net 18)
+	)
+	(segment
 		(start 146.904 76.849)
 		(end 129.421 76.849)
-		(width 0.2)
-		(layer "F.Cu")
-		(net 18)
-	)
-	(segment
-		(start 131.961 124.47676)
-		(end 131.961 119.311)
 		(width 0.2)
 		(layer "F.Cu")
@@
 	)
 	(segment
-		(start 131.28676 125.151)
-		(end 131.961 124.47676)
-		(width 0.2)
-		(layer "F.Cu")
+		(start 126.881 125.151)
+		(end 133.82676 125.151)
+		(width 0.2)
+		(layer "F.Cu")
